File: PCBs/LeftHandV4/LeftHandV4.kicad_pcb (KiCad board)
At the start: 2 copper layers, 343.5 x 150 mm, 83 parts

Commit message: V4 base plates, initial controller PCB.
Parts:
- added SCREW_HOLE: VAL**, SCREW_HOLE, F.Cu at (3.50, 3.50)
- added SCREW_HOLE: VAL**, SCREW_HOLE, F.Cu at (340.0, 3.50)
- added SCREW_HOLE: VAL**, SCREW_HOLE, F.Cu at (172.0, 3.50)
- added SCREW_HOLE: VAL**, SCREW_HOLE, F.Cu at (3.50, 146.5)
- added SCREW_HOLE: VAL**, SCREW_HOLE, F.Cu at (172.0, 146.5)
- added SCREW_HOLE: VAL**, SCREW_HOLE, F.Cu at (340.0, 146.5)
- added SCREW_HOLE: VAL**, SCREW_HOLE, F.Cu at (172.0, 95.0)
- moved LEFT_DSUB1 5.00 mm to (88.5, 7.50)
Changed lines of the file:
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@@
     (links 492)
     (no_connects 492)
-    (area 0 0 0 0)
+    (area -0.050001 -0.050001 343.550001 150.050001)
     (thickness 1.6)
     (drawings 4)
     (tracks 0)
     (zones 0)
-    (modules 83)
+    (modules 90)
     (nets 190)
   )
@@
     (mod_text_size 1 1)
     (mod_text_width 0.15)
-    (pad_size 1.5 1.5)
-    (pad_drill 0.6)
+    (pad_size 2.4 2.4)
+    (pad_drill 2.4)
     (pad_to_mask_clearance 0)
     (aux_axis_origin 0 0)
@@
   )
   (module DB25FD (layer F.Cu)
-    (at 83.5 7.5 180)
+    (at 88.5 7.5 180)
     (descr "Connecteur DB25 femelle droit")
     (tags "CONN DB25")
@@
     )
   )
+  (module SCREW_HOLE (layer F.Cu)
+    (at 3.5 3.5)
+    (fp_text reference SCREW_HOLE (at 0.1 1.95) (layer F.SilkS)
+      (effects (font (size 1 1) (thickness 0.15)))
+    )
+    (fp_text value VAL** (at 0.15 -2.2) (layer F.SilkS)
+      (effects (font (size 1 1) (thickness 0.15)))
+    )
+    (pad HOLE thru_hole circle (at 0 0) (size 2.4 2.4) (drill 2.4)
+      (layers *.Cu *.Mask F.SilkS)
+    )
+  )
+  (module SCREW_HOLE (layer F.Cu)
+    (at 340 3.5)
+    (fp_text reference SCREW_HOLE (at 0.1 1.95) (layer F.SilkS)
+      (effects (font (size 1 1) (thickness 0.15)))
+    )
+    (fp_text value VAL** (at 0.15 -2.2) (layer F.SilkS)
+      (effects (font (size 1 1) (thickness 0.15)))
+    )
+    (pad HOLE thru_hole circle (at 0 0) (size 2.4 2.4) (drill 2.4)
+      (layers *.Cu *.Mask F.SilkS)
+    )
+  )
+  (module SCREW_HOLE (layer F.Cu)
+    (at 172 3.5)
+    (fp_text reference SCREW_HOLE (at 0.1 1.95) (layer F.SilkS)
+      (effects (font (size 1 1) (thickness 0.15)))
+    )
+    (fp_text value VAL** (at 0.15 -2.2) (layer F.SilkS)
+      (effects (font (size 1 1) (thickness 0.15)))
+    )
+    (pad HOLE thru_hole circle (at 0 0) (size 2.4 2.4) (drill 2.4)
+      (layers *.Cu *.Mask F.SilkS)
+    )
+  )
+  (module SCREW_HOLE (layer F.Cu)
+    (at 3.5 146.5)
+    (fp_text reference SCREW_HOLE (at 0.1 1.95) (layer F.SilkS)
+      (effects (font (size 1 1) (thickness 0.15)))
+    )
+    (fp_text value VAL** (at 0.15 -2.2) (layer F.SilkS)
+      (effects (font (size 1 1) (thickness 0.15)))
+    )
+    (pad HOLE thru_hole circle (at 0 0) (size 2.4 2.4) (drill 2.4)
+      (layers *.Cu *.Mask F.SilkS)
+    )
+  )
+  (module SCREW_HOLE (layer F.Cu)
+    (at 172 146.5)
+    (fp_text reference SCREW_HOLE (at 0.1 1.95) (layer F.SilkS)
+      (effects (font (size 1 1) (thickness 0.15)))
+    )
+    (fp_text value VAL** (at 0.15 -2.2) (layer F.SilkS)
+      (effects (font (size 1 1) (thickness 0.15)))
+    )
+    (pad HOLE thru_hole circle (at 0 0) (size 2.4 2.4) (drill 2.4)
+      (layers *.Cu *.Mask F.SilkS)
+    )
+  )
+  (module SCREW_HOLE (layer F.Cu)
+    (at 340 146.5)
+    (fp_text reference SCREW_HOLE (at 0.1 1.95) (layer F.SilkS)
+      (effects (font (size 1 1) (thickness 0.15)))
+    )
+    (fp_text value VAL** (at 0.15 -2.2) (layer F.SilkS)
+      (effects (font (size 1 1) (thickness 0.15)))
+    )
+    (pad HOLE thru_hole circle (at 0 0) (size 2.4 2.4) (drill 2.4)
+      (layers *.Cu *.Mask F.SilkS)
+    )
+  )
+  (module SCREW_HOLE (layer F.Cu)
+    (at 172 95)
+    (fp_text reference SCREW_HOLE (at 0.1 1.95) (layer F.SilkS)
+      (effects (font (size 1 1) (thickness 0.15)))
+    )
+    (fp_text value VAL** (at 0.15 -2.2) (layer F.SilkS)
+      (effects (font (size 1 1) (thickness 0.15)))
+    )
+    (pad HOLE thru_hole circle (at 0 0) (size 2.4 2.4) (drill 2.4)
+      (layers *.Cu *.Mask F.SilkS)
+    )
+  )

Commit message: Left Hand V4 PCB w/ stabilizers.
Parts:
- KEY_L3, NUM_0: footprint SW_DIODE -> SW2_DIODE_R
- LEFT_CONTROL1, LEFT_WIN1: footprint SW_DIODE -> SW_DIODE_RTOP
- LEFT_SHIFT1, LEFT_SPACE1, NUM_ENTER1, NUM_PLUS1: footprint SW_DIODE -> SW2_DIODE_L
- turned NUM_ENTER1 to 270 degrees
- turned NUM_PLUS1 to 270 degrees
Routing:
- net N-000004: track 0.00 -> 2291.3 mm, vias 0 -> 8
- net N-0000062: track 0.00 -> 2284.5 mm, vias 0 -> 1
- net N-00000187: track 0.00 -> 788.3 mm, vias 0 -> 9
- net N-000008: track 0.00 -> 504.0 mm, vias 0 -> 4
- net N-00000186: track 0.00 -> 503.2 mm, vias 0 -> 1
- net N-000007: track 0.00 -> 497.3 mm, vias 0 -> 6
- net N-00000178: track 0.00 -> 449.1 mm, vias 0 -> 2
- net N-000006: track 0.00 -> 437.4 mm, vias 0 -> 4
- net N-00000179: track 0.00 -> 423.0 mm, vias 0 -> 1
- net N-000005: track 0.00 -> 401.3 mm, vias 0 -> 4
- net N-00000176: track 0.00 -> 401.2 mm, vias 0 -> 3
- net N-00000174: track 0.00 -> 387.9 mm, vias 0 -> 2
- net N-00000177: track 0.00 -> 383.6 mm, vias 0 -> 2
- net N-00000189: track 0.00 -> 380.6 mm, vias 0 -> 4
- net N-00000172: track 0.00 -> 370.6 mm, vias 0 -> 3
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