File: PCBs/RightHandV4/RightHandV4.kicad_pcb (KiCad board)
At the start: 2 copper layers, 372 x 150 mm, 96 parts

Commit message: Finished RightHandV4 board and Gerber exports.
Connections:
- MACRO_M4 pad 8: Net-(MACRO_M4-Pad8) -> Net-(DSUB25-Pad25)
- NUM_4 pad 8: Net-(MACRO_M4-Pad8) -> Net-(DSUB25-Pad25)
- NUM_5 pad 8: Net-(MACRO_M4-Pad8) -> Net-(DSUB25-Pad25)
- NUM_6 pad 8: Net-(MACRO_M4-Pad8) -> Net-(DSUB25-Pad25)
Routing:
- net Net-(DSUB25-Pad24): track 0.00 -> 2816.8 mm, vias 0 -> 1
- net Net-(DSUB25-Pad25): track 0.00 -> 2461.9 mm, vias 0 -> 7
- net Net-(DSUB25-Pad11): track 0.00 -> 774.2 mm, vias 0 -> 9
- net Net-(DSUB25-Pad10): track 0.00 -> 653.4 mm, vias 0 -> 6
- net Net-(DSUB25-Pad12): track 0.00 -> 522.6 mm, vias 0 -> 14
- net Net-(DSUB25-Pad21): track 0.00 -> 513.3 mm, vias 0 -> 5
- net Net-(DSUB25-Pad20): track 0.00 -> 442.5 mm, vias 0 -> 1
- net Net-(DSUB25-Pad13): track 0.00 -> 421.1 mm, vias 0 -> 4
- net Net-(DSUB25-Pad22): track 0.00 -> 419.3 mm, vias 0 -> 2
- net Net-(DSUB25-Pad23): track 0.00 -> 403.4 mm, vias 0 -> 4
- net Net-(DSUB25-Pad14): track 0.00 -> 395.9 mm, vias 0 -> 2
- net Net-(DSUB25-Pad8): track 0.00 -> 394.3 mm, vias 0 -> 2
- net Net-(DSUB25-Pad15): track 0.00 -> 369.8 mm, vias 0 -> 2
- net Net-(DSUB25-Pad9): track 0.00 -> 364.5 mm, vias 0 -> 3
- net Net-(DSUB25-Pad16): track 0.00 -> 344.0 mm, vias 0 -> 2
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