File: PCBs/RightHandV4/RightHandV4.sch (KiCad schematic (older format))
At the start: 89 parts

Commit message: Finished RightHandV4 board and Gerber exports.
Connections:
- net at DSUB25.25 (P25), FUNC_F10.8 (GND), FUNC_F11.8 (GND)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: now also MACRO_M4.8 (GND), NUM_4.8 (GND), NUM_5.8 (GND), NUM_6.8 (GND)
Changed lines of the file:
@@
 LIBS:valves
 LIBS:Keyboard
+LIBS:RightHandV4-cache
 EELAYER 25 0
 EELAYER END
@@
 Connection ~ 15750 4550
 Wire Wire Line
-	650  5650 8150 5650
+	650  5650 16700 5650
 Wire Wire Line
 	1500 5650 1500 5600
@@
 Connection ~ 7200 5650
 Wire Wire Line
-	8200 5650 16700 5650
-Wire Wire Line
 	12900 5650 12900 5600
 Wire Wire Line
@@
 	12250 1050 12250 6300
 Connection ~ 12250 6300
+Connection ~ 8150 5650
 $EndSCHEMATC
