File: Mini/V2/PCB/LeftHand.sch (KiCad schematic (older format))
At the start: 30 parts

Commit message: Updating LH PCB register to read 01 for register[4..5] and RH to read 10.  V1 will read as 00 for controller logic backward compatibility.
Parts:
- UDINN9: symbol Mini:MiniDINN9 -> LeftHand-rescue:MiniDINN9-Mini
Connections:
- net GND: no longer UREG1.13 (I2)
- net VCC: now also UREG1.13 (I2)
Changed lines of the file:
@@
 $EndDescr
 $Comp
-L Mini:MiniDINN9 UDINN9
+L LeftHand-rescue:MiniDINN9-Mini UDINN9
 U 1 1 60DBA7F6
 P 9950 5700
@@
 	9750 3200 9850 3200
 Wire Wire Line
-	9350 2650 9550 2650
+	9350 2650 9450 2650
 Wire Wire Line
 	9550 2650 9550 2500
@@
 	8800 1650 8900 1650
 Connection ~ 8800 1550
-Wire Wire Line
-	8800 1650 8800 1750
-Wire Wire Line
-	8800 1750 8900 1750
 Connection ~ 8800 1650
 Wire Wire Line
-	8800 1750 8800 1850
-Wire Wire Line
 	8800 1850 8900 1850
-Connection ~ 8800 1750
 NoConn ~ 10600 1450
 NoConn ~ 7550 5300
@@
 Wire Wire Line
 	7650 1300 7650 2250
+Wire Wire Line
+	8800 1650 8800 1850
+Wire Wire Line
+	8900 1750 9450 1750
+Wire Wire Line
+	9450 1750 9450 2650
+Connection ~ 9450 2650
+Wire Wire Line
+	9450 2650 9550 2650
 $EndSCHEMATC
