File: Mini/V2/PCB/RightHand.sch (KiCad schematic (older format))
At the start: 30 parts

Commit message: Updating LH PCB register to read 01 for register[4..5] and RH to read 10.  V1 will read as 00 for controller logic backward compatibility.
Parts:
- UD9: symbol Mini:MiniDINN9 -> RightHand-rescue:MiniDINN9-Mini
Connections:
- net GND: no longer UREG1.14 (I3)
- net VCC: now also UREG1.14 (I3)
Changed lines of the file:
@@
 $EndDescr
 $Comp
-L Mini:MiniDINN9 UD9
+L RightHand-rescue:MiniDINN9-Mini UD9
 U 1 1 60D91131
 P 9850 5850
@@
 F 3 "" H 10250 3300 50  0001 C CNN
 	1    10200 3550
-	1    0    0    -1
-$EndComp
-$Comp
-L Mini:ParallelLoadShiftRegister UREG1
-U 1 1 60D92831
-P 10250 1250
-F 0 "UREG1" H 10200 111 50  0000 C CNN
-F 1 "ParallelLoadShiftRegister" H 10200 20  50  0000 C CNN
-F 2 "Mini:DualInlineMicrochip2x8" H 10250 1250 50  0001 C CNN
-F 3 "" H 10250 1250 50  0001 C CNN
-	1    10250 1250
 	1    0    0    -1
 $EndComp
@@
 Connection ~ 10100 2700
 Wire Wire Line
-	9800 2400 10000 2400
+	9800 2400 9900 2400
 Wire Wire Line
 	10000 2400 10000 2300
@@
 	9300 1550 9350 1550
 Connection ~ 9300 1450
-Wire Wire Line
-	9300 1550 9300 1650
-Wire Wire Line
-	9300 1650 9350 1650
-Connection ~ 9300 1550
 Text GLabel 9100 1150 0    50   Input ~ 0
 SH_LD
@@
 	4200 2250 4200 3400
 Connection ~ 4200 3400
+$Comp
+L Mini:ParallelLoadShiftRegister UREG1
+U 1 1 60D92831
+P 10250 1250
+F 0 "UREG1" H 10200 111 50  0000 C CNN
+F 1 "ParallelLoadShiftRegister" H 10200 20  50  0000 C CNN
+F 2 "Mini:DualInlineMicrochip2x8" H 10250 1250 50  0001 C CNN
+F 3 "" H 10250 1250 50  0001 C CNN
+	1    10250 1250
+	1    0    0    -1
+$EndComp
+Wire Wire Line
+	9350 1650 9900 1650
+Wire Wire Line
+	9900 1650 9900 2400
+Connection ~ 9900 2400
+Wire Wire Line
+	9900 2400 10000 2400
 $EndSCHEMATC
